File: PCB/RYZEE/GBA_EMU.brd (EAGLE design)
At the start: 130.7 x 72.9 mm, 14 parts, among them J1 SWTCHCRFT_3.5JACK5-JACK-SMD, SW1 LEFT, SW2 RIGHT, SW3 PWR_SWITCH, U1 RPI-ZEROSMD, U3 LM4875

Commit message: cleaned pcb
removed most parts and marked positions
Parts:
- removed J1: SWTCHCRFT_3.5JACK5-JACK-SMD, gba-zero-parts:4-JACK-SMD
- removed R1: 27k, GBA:VOLUME
- removed R2: RK10J12E0A0A, gba-zero-parts:RK10J12E0A0A
- removed S3: SHOULDER_BUTTON, gba-zero-parts:SHOULDER_BUTTON
- removed S4: PWR_SWITCH, gba-zero-parts:PWR-SWITCH
- removed S5: D-PAD, gba-zero-parts:D-PAD
- removed S6: AB_BUTTON, gba-zero-parts:AB_BUTTON
- removed SW1: LEFT, GBA:BUMPER
- removed SW2: RIGHT, GBA:BUMPER
- removed SW3: PWR_SWITCH, GBA:PWR_SWITCH
- removed U1: RPI-ZEROSMD, gba-zero-parts:RPI-SMD
- removed U3: LM4875, gba-zero-parts:SO-8
- S1: value START_SELECT_BUTTON -> SHOULDER_BUTTON; device gba-zero-parts:START_SELECT_BUTTON -> gba-zero-parts:SHOULDER_BUTTON
- moved S2 108.7 mm to (122.8, 9.19), turned to 350 degrees
- moved S1 5.98 mm to (9.54, 9.43), turned to 10 degrees
Connections:
- removed net 3.3V: U1.1
- removed net 5V: U1.2, U1.4
- removed net A_BTN: U1.35
- removed net B_BTN: U1.37
- removed net DOWN: U1.11
- removed net GND: U1.14, U1.20, U1.25, U1.30, U1.34, U1.39, U1.6, U3.6
- removed net LEFT: U1.13
- removed net LEFT_BUMP: U1.31
- removed net PWM0: U1.12
- removed net RIGHT: U1.15
- removed net RIGHT_BUMP: U1.40
- removed net RXD: U1.8
- removed net SELECT: U1.18
- removed net START: U1.16
- removed net TFT_CS: U1.24
- removed net TFT_DC: U1.5
- removed net TFT_LED: U1.7
- removed net TFT_MOSI: U1.19
- removed net TFT_RESET: U1.3
- removed net TFT_SCK: U1.23
- removed net TXD: U1.10
- removed net UP: U1.29
- removed net VDD: U3.1
