File: PCB/RYZEE/GBA_EMU.sch (EAGLE design)
At the start: 14 parts, among them J1 SWTCHCRFT_3.5JACK5-JACK-SMD, SW1 LEFT, SW2 RIGHT, SW3 PWR_SWITCH, U1 RPI-ZEROSMD, U3 LM4875

Commit message: cleaned pcb
removed most parts and marked positions
Parts:
- removed J1: SWTCHCRFT_3.5JACK5-JACK-SMD, gba-zero-parts:SWTCHCRFT_3.5JACK5-JACK-SMD
- removed R1: 27k, GBA:VOLUME
- removed R2: RK10J12E0A0A, gba-zero-parts:RK10J12E0A0A
- removed S3: SHOULDER_BUTTON, gba-zero-parts:SHOULDER_BUTTON
- removed S4: PWR_SWITCH, gba-zero-parts:PWR_SWITCH
- removed S5: D-PAD, gba-zero-parts:D-PAD
- removed S6: AB_BUTTON, gba-zero-parts:AB_BUTTON
- removed SW1: LEFT, GBA:BUTTON
- removed SW2: RIGHT, GBA:BUTTON
- removed SW3: PWR_SWITCH, GBA:PWR_SWITCH
- removed U1: RPI-ZEROSMD, gba-zero-parts:RPI-ZEROSMD
- removed U3: LM4875, gba-zero-parts:LM4875
- S1: value START_SELECT_BUTTON -> SHOULDER_BUTTON; device gba-zero-parts:START_SELECT_BUTTON -> gba-zero-parts:SHOULDER_BUTTON
Connections:
- removed net 3.3V: U1.3.3V@1
- removed net 5V: U1.5.0V@1, U1.5.0V@2
- removed net A_BTN: U1.GPIO19
- removed net B_BTN: U1.GPIO26
- removed net DOWN: U1.GPIO17
- removed net GND: U1.GND@2, U1.GND@3, U1.GND@4, U1.GND@5, U1.GND@6, U1.GND@7, U1.GND@8
- removed net LEFT: U1.GPIO27
- removed net LEFT_BUMP: U1.GPIO6
- removed net PWM0: U1.GPIO18
- removed net RIGHT: U1.GPIO22
- removed net RIGHT_BUMP: U1.GPIO21
- removed net RXD: U1.TXD
- removed net SELECT: U1.GPIO24
- removed net START: U1.GPIO23
- removed net TFT_CS: U1.#SPI_CE0
- removed net TFT_DC: U1.SCL
- removed net TFT_LED: U1.GPIO4
- removed net TFT_MOSI: U1.SPI_MOSI
- removed net TFT_RESET: U1.SDA
- removed net TFT_SCK: U1.SPI_SCLK
- removed net TXD: U1.RXD
- removed net UP: U1.GPIO5
Other:
- moved on the sheet: S2
