File: PCB/KiCAD/GBA_EMU.kicad_pcb (KiCad board)
At the start: 2 copper layers, 130.7 x 72.9 mm, 18 parts, among them J1 Raspberry_Pi_2_3

Commit message: LCD Connection
https://github.com/juj/fbcp-ili9341#if-you-wired-the-display-to-the-pi-yourself

https://sudomod.com/forum/viewtopic.php?f=22&t=5854

Screen<------------>Raspberry Pi 3 or zero
LED<-------------->Pin 12 (GPIO18)
SCK<-------------->Pin 23 (GPIO11)
SDI(MOSI)<----->Pin 19 (GPIO10)
DC<--------------->Pin 22 (GPIO24)
RESET<----------->Pin 26 (GPIO25)
CS<----------------->Pin 24 (GPIO8)
Connections:
- net Net-(J1-Pad12) renamed TFT_LED
- net Net-(J1-Pad18) renamed TFT_DC
- net Net-(J1-Pad22) renamed TFT_RESET

Commit message: Audio, LCD, Buttons
Parts:
- added U1: ILI3941, GBA_EMU:18PIN-0.8MM, F.Cu at (114.0, 101.0)
- J1: footprint Module:Raspberry_Pi_Zero_Socketed_THT_FaceDown_MountingHoles -> GBA_EMU:Raspberry_Pi_Zero_Socketed_THT_FaceDown_MountingHoles
- moved J1 1.52 mm to (172.7, 103.1)
Connections:
- J1 pad 1: Net-(J1-Pad1) -> +3V3
- J1 pad 12: TFT_LED -> PWM_Mono
- J1 pad 17: Net-(J1-Pad17) -> +3V3
- J1 pad 21: Net-(J1-Pad21) -> TFT_MISO
- J1 pad 33: Net-(J1-Pad33) -> TFT_LED
